File: hw/videoadc.sch (KiCad schematic (older format))
At the start: 56 parts, among them P1 CONN_4X2, P2 CONN_20X2, U1 LM358

Commit message: tweaks tweaks tweaks
also updated the schematic with actual values
Parts:
- R6, R7, R8, R9: value 120 -> 470
- RV1, RV2, RV3, RV4: value 10K -> 100K
Changed lines of the file:
@@
 LIBS:contrib
 LIBS:valves
+LIBS:videoadc-cache
 EELAYER 24 0
 EELAYER END
@@
 P 5650 4200
 F 0 "RV1" H 5650 4100 50  0000 C CNN
-F 1 "10K" H 5650 4200 50  0000 C CNN
+F 1 "100K" H 5650 4200 50  0000 C CNN
 F 2 "" H 5650 4200 60  0000 C CNN
 F 3 "" H 5650 4200 60  0000 C CNN
@@
 P 6400 4200
 F 0 "RV2" H 6400 4100 50  0000 C CNN
-F 1 "10K" H 6400 4200 50  0000 C CNN
+F 1 "100K" H 6400 4200 50  0000 C CNN
 F 2 "" H 6400 4200 60  0000 C CNN
 F 3 "" H 6400 4200 60  0000 C CNN
@@
 P 7150 4200
 F 0 "RV3" H 7150 4100 50  0000 C CNN
-F 1 "10K" H 7150 4200 50  0000 C CNN
+F 1 "100K" H 7150 4200 50  0000 C CNN
 F 2 "" H 7150 4200 60  0000 C CNN
 F 3 "" H 7150 4200 60  0000 C CNN
@@
 P 7900 4200
 F 0 "RV4" H 7900 4100 50  0000 C CNN
-F 1 "10K" H 7900 4200 50  0000 C CNN
+F 1 "100K" H 7900 4200 50  0000 C CNN
 F 2 "" H 7900 4200 60  0000 C CNN
 F 3 "" H 7900 4200 60  0000 C CNN
@@
 P 7000 1250
 F 0 "R6" V 7080 1250 40  0000 C CNN
-F 1 "120" V 7007 1251 40  0000 C CNN
+F 1 "470" V 7007 1251 40  0000 C CNN
 F 2 "" V 6930 1250 30  0000 C CNN
 F 3 "" H 7000 1250 30  0000 C CNN
@@
 P 7000 1850
 F 0 "R7" V 7080 1850 40  0000 C CNN
-F 1 "120" V 7007 1851 40  0000 C CNN
+F 1 "470" V 7007 1851 40  0000 C CNN
 F 2 "" V 6930 1850 30  0000 C CNN
 F 3 "" H 7000 1850 30  0000 C CNN
@@
 P 7000 2500
 F 0 "R8" V 7080 2500 40  0000 C CNN
-F 1 "120" V 7007 2501 40  0000 C CNN
+F 1 "470" V 7007 2501 40  0000 C CNN
 F 2 "" V 6930 2500 30  0000 C CNN
 F 3 "" H 7000 2500 30  0000 C CNN
@@
 P 7000 3100
 F 0 "R9" V 7080 3100 40  0000 C CNN
-F 1 "120" V 7007 3101 40  0000 C CNN
+F 1 "470" V 7007 3101 40  0000 C CNN
 F 2 "" V 6930 3100 30  0000 C CNN
 F 3 "" H 7000 3100 30  0000 C CNN

Commit message: schematic fluff
Parts:
- C1, C10, C11, C12, C13, C14, C6, C7, C8, C9: symbol C -> C-RESCUE-videoadc
- C2, C3, C4, C5: symbol CP1 -> CP1-RESCUE-videoadc
- R1, R11, R2, R3, R4, R5, R6, R7, R8, R9: symbol R -> R-RESCUE-videoadc
